File: Platine/HM-LC-Sw1-Pl-DN-R1_S26.kicad_pcb (KiCad board)
At the start: 2 copper layers, 20.1 x 29.7 mm, 13 parts, among them J1 FTDI, J3 Reset, J4 Conn_01x06_Female, U1 ATmega328P-AU, U2 CC1101-

Commit message: update to V1.1
Parts:
- C1, C2, C3, C4, C5: footprint Capacitor_SMD:C_0603_1608Metric_Pad1.05x0.95mm_HandSolder -> Capacitor_SMD:C_0805_2012Metric_Pad1.15x1.40mm_HandSolder
- J1: footprint Connector_PinHeader_2.54mm:PinHeader_1x05_P2.54mm_Vertical -> Connector_PinHeader_2.54mm:PinHeader_1x06_P2.54mm_Vertical
- J3: footprint Connector_Pin:Pin_D0.7mm_L6.5mm_W1.8mm_FlatFork -> Connector_PinHeader_2.00mm:PinHeader_1x01_P2.00mm_Vertical
- R1: footprint Capacitor_SMD:C_0603_1608Metric_Pad1.05x0.95mm_HandSolder -> Resistor_SMD:R_0805_2012Metric_Pad1.15x1.40mm_HandSolder
- moved J1 2.45 mm to (146.8, 95.7)
- moved C4 1.81 mm to (148.8, 102.0), turned to 270 degrees
- moved R1 1.14 mm to (146.8, 104.1), turned to 90 degrees
- moved C5 0.95 mm to (147.9, 117.7)
- moved J3 0.56 mm to (147.3, 98.4)
- moved C1 0.54 mm to (159.8, 110.8)
- moved C2 0.51 mm to (156.9, 105.0)
Connections:
- net /SCK renamed /SCLK
- J1 pad 2: /RXD -> /TXD
- J1 pad 3: /TXD -> /RXD
Routing:
- net VCC: track 46.2 -> 79.9 mm
- net GND: track 49.4 -> 21.9 mm, vias 0 -> 13
- net /GDO0: track 23.2 -> 30.3 mm, vias 1 -> 2
- net /TXD: track 11.5 -> 17.0 mm
- net /LED(J5): track 10.3 -> 6.65 mm
- net /SCLK: track 7.52 -> 10.5 mm
- net /BUTTON(J4): track 18.2 -> 20.3 mm
- net /DTR: track 3.95 -> 5.76 mm
- net /CSN: track 10.2 -> 11.5 mm
- net /Reset: track 11.0 -> 12.3 mm
- net /MOSI: track 12.4 -> 13.0 mm
- added copper zone on F.Cu, net GND
- removed copper zone on F.Cu, net VCC
Other:
- outline, holes or cut-outs redrawn
- board text added: "Ant: 83mm"
- board text added: "v1.1 - 01/20 P.Wulfert"
- board text removed: "v1.0 - 01/19 P.Wulfert"
